File: kicad/Yaxis.sch (KiCad schematic (older format))
At the start: 16 parts, among them P14 \"1791-ZL262-8SG\", P15 \"1791-ZL262-8SG\", Q3 IRLR2905ZPBF, U1 \"1815-CD40109BPWR\"

Commit message: Draw schematic
Commit before trying newer version of KiCad
Connections:
- wire segments 59 -> 50
Changed lines of the file:
@@
 LIBS:opto
 LIBS:transistor
+LIBS:conn
 LIBS:RAMPS_plus-cache
 EELAYER 27 0
@@
 	2000 5350 2200 5350
 Wire Wire Line
-	1900 5450 2000 5450
-Wire Wire Line
-	2000 5450 2200 5450
+	1900 5450 2200 5450
 Wire Wire Line
 	2200 5550 1900 5550
@@
 	2900 6050 3200 6050
 Wire Wire Line
-	3200 5450 3200 6050
-Wire Wire Line
-	3200 6050 3200 6250
+	3200 5450 3200 6250
 Wire Wire Line
 	2900 5450 3200 5450
@@
 Stepper Driver
 $Comp
-L +12V #PWR36
+L +12V #PWR045
 U 1 1 534EC799
 P 3200 4950
-F 0 "#PWR36" H 3200 4900 20  0001 C CNN
+F 0 "#PWR045" H 3200 4900 20  0001 C CNN
 F 1 "+12V" H 3200 5100 60  0000 C CNN
 F 2 "~" H 3200 4950 60  0000 C CNN
@@
 	3400 5950 3400 5100
 $Comp
-L +5V #PWR38
+L +5V #PWR046
 U 1 1 534EC79A
 P 3400 5100
-F 0 "#PWR38" H 3400 5190 20  0001 C CNN
+F 0 "#PWR046" H 3400 5190 20  0001 C CNN
 F 1 "+5V" H 3390 5240 60  0000 C CNN
 F 2 "~" H 3400 5100 60  0000 C CNN
@@
 $EndComp
 $Comp
-L GND #PWR37
+L GND #PWR047
 U 1 1 53470080
 P 3200 6250
-F 0 "#PWR37" H 3200 6250 30  0001 C CNN
+F 0 "#PWR047" H 3200 6250 30  0001 C CNN
 F 1 "GND" H 3200 6180 30  0001 C CNN
 F 2 "~" H 3200 6250 60  0000 C CNN
@@
 $EndComp
 $Comp
-L +12V #PWR34
+L +12V #PWR048
 U 1 1 53470091
 P 2700 6550
-F 0 "#PWR34" H 2700 6500 20  0001 C CNN
+F 0 "#PWR048" H 2700 6500 20  0001 C CNN
 F 1 "+12V" H 2700 6700 60  0000 C CNN
 F 2 "~" H 2700 6550 60  0000 C CNN
@@
 $EndComp
 $Comp
-L GND #PWR35
+L GND #PWR049
 U 1 1 53470097
 P 2700 7150
-F 0 "#PWR35" H 2700 7150 30  0001 C CNN
+F 0 "#PWR049" H 2700 7150 30  0001 C CNN
 F 1 "GND" H 2700 7080 30  0001 C CNN
 F 2 "~" H 2700 7150 60  0000 C CNN
@@
 	2700 6550 2700 6650
 $Comp
-L +5V #PWR32
+L +5V #PWR050
 U 1 1 534700AA
 P 2000 4650
-F 0 "#PWR32" H 2000 4740 20  0001 C CNN
+F 0 "#PWR050" H 2000 4740 20  0001 C CNN
 F 1 "+5V" H 1990 4790 60  0000 C CNN
 F 2 "~" H 2000 4650 60  0000 C CNN
@@
 $EndComp
 Wire Wire Line
-	2000 5150 2000 5250
-Wire Wire Line
-	2000 5250 2000 5350
+	2000 5150 2000 5350
 Wire Wire Line
 	1150 5250 2000 5250
@@
 Connection ~ 2000 5450
 $Comp
-L GND #PWR33
+L GND #PWR051
 U 1 1 534700CA
 P 2000 7150
-F 0 "#PWR33" H 2000 7150 30  0001 C CNN
+F 0 "#PWR051" H 2000 7150 30  0001 C CNN
 F 1 "GND" H 2000 7080 30  0001 C CNN
 F 2 "~" H 2000 7150 60  0000 C CNN
@@
 	2000 7150 2000 7050
 $Comp
-L +5V #PWR31
+L +5V #PWR052
 U 1 1 534700D1
 P 1300 5000
-F 0 "#PWR31" H 1300 5090 20  0001 C CNN
+F 0 "#PWR052" H 1300 5090 20  0001 C CNN
 F 1 "+5V" H 1290 5140 60  0000 C CNN
 F 2 "~" H 1300 5000 60  0000 C CNN
@@
 	1300 5650 1400 5650
 Wire Wire Line
-	1300 5000 1300 5450
-Wire Wire Line
-	1300 5450 1300 5550
-Wire Wire Line
-	1300 5550 1300 5650
+	1300 5000 1300 5650
 Wire Wire Line
 	1400 5450 1300 5450
@@
 Y
 $Comp
-L GND #PWR43
+L GND #PWR053
 U 1 1 534EC7A3
 P 6550 6300
-F 0 "#PWR43" H 6550 6300 30  0001 C CNN
+F 0 "#PWR053" H 6550 6300 30  0001 C CNN
 F 1 "GND" H 6550 6230 30  0001 C CNN
 F 2 "~" H 6550 6300 60  0000 C CNN
@@
 D8
 Wire Wire Line
-	4900 6150 5050 6150
-Wire Wire Line
-	5050 6150 5200 6150
-$Comp
-L VCC #PWR42
+	4900 6150 5200 6150
+$Comp
+L VCC #PWR054
 U 1 1 534D8FF4
 P 5500 5850
-F 0 "#PWR42" H 5500 5800 20  0001 C CNN
+F 0 "#PWR054" H 5500 5800 20  0001 C CNN
 F 1 "VCC" H 5500 6000 60  0000 C CNN
 F 2 "~" H 5500 5850 60  0000 C CNN
@@
 $EndComp
 $Comp
-L GND #PWR41
+L GND #PWR055
 U 1 1 534D9642
 P 5050 6750
-F 0 "#PWR41" H 5050 6750 30  0001 C CNN
+F 0 "#PWR055" H 5050 6750 30  0001 C CNN
 F 1 "GND" H 5050 6680 30  0001 C CNN
 F 2 "~" H 5050 6750 60  0000 C CNN
@@
 $EndComp
 $Comp
-L GND #PWR40
+L GND #PWR056
 U 1 1 534ECB96
 P 5000 4050
-F 0 "#PWR40" H 5000 4050 30  0001 C CNN
+F 0 "#PWR056" H 5000 4050 30  0001 C CNN
 F 1 "GND" H 5000 3980 30  0001 C CNN
 F 2 "~" H 5000 4050 60  0000 C CNN
@@
 	5000 4050 5000 4000
 Wire Wire Line
-	5000 3600 5000 3500
-Wire Wire Line
-	5000 3500 5000 3400
-$Comp
-L VCC #PWR39
+	5000 3400 5000 3600
+$Comp
+L VCC #PWR057
 U 1 1 534ECC20
 P 5000 2900
-F 0 "#PWR39" H 5000 2850 20  0001 C CNN
+F 0 "#PWR057" H 5000 2850 20  0001 C CNN
 F 1 "VCC" H 5000 3050 60  0000 C CNN
 F 2 "~" H 5000 2900 60  0000 C CNN
@@
 A15
 Wire Wire Line
-	4900 3500 5000 3500
-Wire Wire Line
-	5000 3500 5400 3500
+	4900 3500 5400 3500
 Connection ~ 5000 3500
 $Comp
@@
 $EndComp
 $Comp
-L VCC #PWR47
+L VCC #PWR058
 U 1 1 534ED3AF
 P 8350 5300
-F 0 "#PWR47" H 8350 5250 20  0001 C CNN
+F 0 "#PWR058" H 8350 5250 20  0001 C CNN
 F 1 "VCC" H 8350 5450 60  0000 C CNN
 F 2 "~" H 8350 5300 60  0000 C CNN
@@
 $EndComp
 $Comp
-L +12V #PWR49
+L +12V #PWR059
 U 1 1 534ED3B5
 P 8550 5300
-F 0 "#PWR49" H 8550 5250 20  0001 C CNN
+F 0 "#PWR059" H 8550 5250 20  0001 C CNN
 F 1 "+12V" H 8550 5450 60  0000 C CNN
 F 2 "~" H 8550 5300 60  0000 C CNN
@@
 $EndComp
 $Comp
-L GND #PWR48
+L GND #PWR060
 U 1 1 534ED3BB
 P 8450 6100
-F 0 "#PWR48" H 8450 6100 30  0001 C CNN
+F 0 "#PWR060" H 8450 6100 30  0001 C CNN
 F 1 "GND" H 8450 6030 30  0001 C CNN
 F 2 "~" H 8450 6100 60  0000 C CNN
@@
 $EndComp
 $Comp
-L GND #PWR51
+L GND #PWR061
 U 1 1 534ED3D4
 P 9050 6100
-F 0 "#PWR51" H 9050 6100 30  0001 C CNN
+F 0 "#PWR061" H 9050 6100 30  0001 C CNN
 F 1 "GND" H 9050 6030 30  0001 C CNN
 F 2 "~" H 9050 6100 60  0000 C CNN
@@
 $EndComp
 $Comp
-L GND #PWR45
+L GND #PWR062
 U 1 1 534ED3DA
 P 7850 6100
-F 0 "#PWR45" H 7850 6100 30  0001 C CNN
+F 0 "#PWR062" H 7850 6100 30  0001 C CNN
 F 1 "GND" H 7850 6030 30  0001 C CNN
 F 2 "~" H 7850 6100 60  0000 C CNN
@@
 	9050 6100 9050 5950
 $Comp
-L +12V #PWR50
+L +12V #PWR063
 U 1 1 534ED3E2
 P 9050 5300
-F 0 "#PWR50" H 9050 5250 20  0001 C CNN
+F 0 "#PWR063" H 9050 5250 20  0001 C CNN
 F 1 "+12V" H 9050 5450 60  0000 C CNN
 F 2 "~" H 9050 5300 60  0000 C CNN
@@
 $EndComp
 $Comp
-L VCC #PWR44
+L VCC #PWR064
 U 1 1 534ED3E8
 P 7850 5300
-F 0 "#PWR44" H 7850 5250 20  0001 C CNN
+F 0 "#PWR064" H 7850 5250 20  0001 C CNN
 F 1 "VCC" H 7850 5450 60  0000 C CNN
 F 2 "~" H 7850 5300 60  0000 C CNN
@@
 	9050 5300 9050 5550
 $Comp
-L VCC #PWR46
+L VCC #PWR065
 U 1 1 534ED3F0
 P 8200 3950
-F 0 "#PWR46" H 8200 3900 20  0001 C CNN
+F 0 "#PWR065" H 8200 3900 20  0001 C CNN
 F 1 "VCC" H 8200 4100 60  0000 C CNN
 F 2 "~" H 8200 3950 60  0000 C CNN
@@
 	8600 4000 8200 4000
 Wire Wire Line
-	8200 3950 8200 4000
-Wire Wire Line
-	8200 4000 8200 4350
+	8200 3950 8200 4350
 Wire Wire Line
 	8200 4350 8300 4350

Commit message: Change components to my own
References: #1 #19
Parts:
- removed C4: \"1795-EEEFK1V101XP\", 7408hacks/dnxpf, symbol "1795-EEEFK1V101XP"
- added C?: 100u/35V, symbol Cpol
- renumbered C5 to C10, C6 to C11, C7 to C12, D1 to D8, JP4 to JP5, P14 to P10, P15 to P11, R15 to R17, R11 to R18, R16 to R19, R14 to R20, R13 to R21, R12 to R22
Connections:
- wire segments 50 -> 62
Other:
- moved on the sheet: R17
