File: kicad/RAMPS_plus.sch (KiCad schematic (older format))
At the start: 8 parts, among them CON1 CON10, CON2 CON8, CON3 CON8, CON4 CON8, CON6 CON8, CON7 CON8, CON8 CON18x2

Commit message: Place components
Parts:
- gave numbers to parts that had none: 1
Changed lines of the file:
@@
 $EndSheet
 $Comp
-L ArduinoMegaShield MECH?
+L ArduinoMegaShield MECH1
 U 1 1 539B6D78
 P 2200 7200
-F 0 "MECH?" H 2150 7300 60  0000 C CNN
+F 0 "MECH1" H 2150 7300 60  0000 C CNN
 F 1 "ArduinoMegaShield" H 2150 7100 60  0000 C CNN
 F 2 "" H 2100 7200 60  0000 C CNN

Commit message: Add bed connector. Routing.
Connections:
- no-connect marks 6 -> 13
Changed lines of the file:
@@
 	1    0    0    -1
 $EndComp
+NoConn ~ 1750 2600
+NoConn ~ 1750 2700
+NoConn ~ 1750 2800
+NoConn ~ 1750 3800
+NoConn ~ 2650 2900
+NoConn ~ 2650 3000
+NoConn ~ 2000 4600
 $EndSCHEMATC

Commit message: Fix panel connections. Place.
Changed lines of the file:
@@
 $EndComp
 $Comp
-L GND #PWR1
+L GND #PWR01
 U 1 1 536FA4F6
 P 1300 2000
-F 0 "#PWR1" H 1300 2000 30  0001 C CNN
+F 0 "#PWR01" H 1300 2000 30  0001 C CNN
 F 1 "GND" H 1300 1930 30  0001 C CNN
 F 2 "" H 1300 2000 60  0000 C CNN
@@
 $EndComp
 $Comp
-L GND #PWR3
+L GND #PWR02
 U 1 1 536FA739
 P 2550 6400
-F 0 "#PWR3" H 2550 6400 30  0001 C CNN
+F 0 "#PWR02" H 2550 6400 30  0001 C CNN
 F 1 "GND" H 2550 6330 30  0001 C CNN
 F 2 "" H 2550 6400 60  0000 C CNN
@@
 $EndComp
 $Comp
-L GND #PWR2
+L GND #PWR03
 U 1 1 536FA866
 P 1850 6400
-F 0 "#PWR2" H 1850 6400 30  0001 C CNN
+F 0 "#PWR03" H 1850 6400 30  0001 C CNN
 F 1 "GND" H 1850 6330 30  0001 C CNN
 F 2 "" H 1850 6400 60  0000 C CNN
@@
 	1    0    0    -1
 $EndComp
-NoConn ~ 1750 2600
-NoConn ~ 1750 2700
+NoConn ~ 2650 4000
+NoConn ~ 2650 4100
 NoConn ~ 1750 2800
 NoConn ~ 1750 3800

Commit message: Route.
Connections:
- net 5V is gone; now on net +5V: CON8.1, CON8.2
Changed lines of the file:
@@
 $EndComp
 Text GLabel 1850 4500 0    50   UnSpc ~ 0
-5V
++5V
 Text GLabel 2550 4500 2    50   UnSpc ~ 0
-5V
++5V
 NoConn ~ 1750 1200
 NoConn ~ 2650 1000

Commit message: Swap pins
Connections:
- no-connect marks 13 -> 8
Changed lines of the file:
@@
 	1    0    0    -1
 $EndComp
-NoConn ~ 2650 4000
-NoConn ~ 2650 4100
-NoConn ~ 1750 2800
-NoConn ~ 1750 3800
 NoConn ~ 2650 2900
 NoConn ~ 2650 3000
-NoConn ~ 2000 4600
 $EndSCHEMATC

Commit message: Add AGND. Route.
close #27
Connections:
- net +5V: no longer CON2.5
- net GND: no longer CON8.35, CON8.36
- new net AGND: CON8.35, CON8.36
- no-connect marks 8 -> 9
Other:
- note added: "+5V"
Changed lines of the file:
@@
 Text GLabel 1550 1500 0    50   UnSpc ~ 0
 +3V3
-Text GLabel 1550 1600 0    50   UnSpc ~ 0
-+5V
 Text GLabel 1550 2300 0    50   BiDi ~ 0
 A0
@@
 	1    0    0    -1
 $EndComp
-$Comp
-L GND #PWR02
-U 1 1 536FA739
-P 2550 6400
-F 0 "#PWR02" H 2550 6400 30  0001 C CNN
-F 1 "GND" H 2550 6330 30  0001 C CNN
-F 2 "" H 2550 6400 60  0000 C CNN
-F 3 "" H 2550 6400 60  0000 C CNN
-	1    2550 6400
-	1    0    0    -1
-$EndComp
-$Comp
-L GND #PWR03
-U 1 1 536FA866
-P 1850 6400
-F 0 "#PWR03" H 1850 6400 30  0001 C CNN
-F 1 "GND" H 1850 6330 30  0001 C CNN
-F 2 "" H 1850 6400 60  0000 C CNN
-F 3 "" H 1850 6400 60  0000 C CNN
-	1    1850 6400
-	1    0    0    -1
-$EndComp
 Text GLabel 1850 4500 0    50   UnSpc ~ 0
 +5V
@@
 	1550 1500 1750 1500
 Wire Wire Line
-	1550 1600 1750 1600
-Wire Wire Line
 	1300 1700 1750 1700
 Wire Wire Line
@@
 NoConn ~ 2650 2900
 NoConn ~ 2650 3000
+NoConn ~ 1750 1600
+Text Notes 1400 1625 0    50   Italic 0
++5V
+Wire Wire Line
+	2550 6400 1550 6400
+Connection ~ 1850 6400
+Text GLabel 1550 6400 0    50   UnSpc ~ 0
+AGND
 $EndSCHEMATC
