File: kicad/power.sch (KiCad schematic (older format))
At the start: 32 parts, among them CON23 PS-ON, CON24 CON6, CON25 FAN, CON26 Chamber, Q7 FDC6401N, Q8 FDC6401N, Q9 FDC6401N

Commit message: Route.
Connections:
- net A3: now also Q9.3 (G); no longer Q9.1 (G)
- net A4: now also Q9.1 (G); no longer Q9.3 (G)
- net Chamber-fan: now also Q9.6 (D); no longer Q9.4 (D)
- net Chamber-heater: now also Q9.4 (D); no longer Q9.6 (D)
Other:
- moved on the sheet: Q9A, Q9B
Changed lines of the file:
@@
 L FDC6401N Q9
 U 1 1 5394A1D2
+P 7450 2750
+F 0 "Q9" H 7630 2820 60  0000 L CNN
+F 1 "FDC6401N" H 7630 2740 60  0000 L CNN
+F 2 "SOT23-6" H 7630 2670 40  0000 L CNN
+F 3 "" H 7450 2700 60  0000 C CNN
+	1    7450 2750
+	1    0    0    -1
+$EndComp
+$Comp
+L FDC6401N Q9
+U 2 1 5394A1D8
 P 7450 1500
 F 0 "Q9" H 7630 1570 60  0000 L CNN
@@
 F 2 "SOT23-6" H 7630 1420 40  0000 L CNN
 F 3 "" H 7450 1450 60  0000 C CNN
-	1    7450 1500
+	2    7450 1500
 	1    0    0    -1
 $EndComp
-$Comp
-L FDC6401N Q9
-U 2 1 5394A1D8
-P 7450 2750
-F 0 "Q9" H 7630 2820 60  0000 L CNN
-F 1 "FDC6401N" H 7630 2740 60  0000 L CNN
-F 2 "SOT23-6" H 7630 2670 40  0000 L CNN
-F 3 "" H 7450 2700 60  0000 C CNN
-	2    7450 2750
-	1    0    0    -1
-$EndComp

Commit message: Swap pins
Connections:
- net A3 renamed D24
- net A4 renamed D26
Changed lines of the file:
@@
 Text GLabel 4750 1900 0    60   UnSpc ~ 0
 +12V
-Text GLabel 4350 2700 0    50   Input Italic 0
+Text GLabel 4350 2700 0    50   Input ~ 0
 D12
 Wire Wire Line
@@
 Wire Wire Line
 	4650 3950 4350 3950
-Text GLabel 4350 3950 0    50   Input Italic 0
+Text GLabel 4350 3950 0    50   Input ~ 0
 D11
 Text Notes 5050 4150 0    60   Italic 0
@@
 Wire Wire Line
 	3950 6200 3550 6200
-Text GLabel 3550 6200 0    50   Input Italic 0
+Text GLabel 3550 6200 0    50   Input ~ 0
 D47
 $Comp
@@
 Text GLabel 7100 800  0    60   UnSpc ~ 0
 +12V
-Text GLabel 7050 1600 0    50   Input Italic 0
-A3
+Text GLabel 7050 1600 0    50   Input ~ 0
+D24
 Wire Wire Line
 	7550 1200 7550 1300
@@
 Wire Wire Line
 	7350 2850 7050 2850
-Text GLabel 7050 2850 0    50   Input Italic 0
-A4
+Text GLabel 7050 2850 0    50   Input ~ 0
+D26
 Text Notes 7750 3050 0    60   Italic 0
 Power supply fan

Commit message: Pin swap. Route.
Connections:
- net A11: now also C21.1, CON26.6, R30.2; no longer C23.1, CON26.10, R32.2
- net A9: now also C23.1, CON26.10, R32.2; no longer C21.1, CON26.6, R30.2
- net A10 renamed A13
Changed lines of the file:
@@
 $EndComp
 Text GLabel 7100 3950 0    50   Input ~ 0
-A9
+A11
 Text Label 8150 3950 2    60   ~ 0
 ThermC1
@@
 $EndComp
 Text GLabel 8950 3950 0    50   Input ~ 0
-A10
+A13
 Text Label 10000 3950 2    60   ~ 0
 ThermC2
@@
 $EndComp
 Text GLabel 8950 2700 0    50   Input ~ 0
-A11
+A9
 Text Label 10000 2700 2    60   ~ 0
 ThermC3

Commit message: Add AGND. Route.
close #27
Connections:
- net GND: no longer C21.2, C22.2, C23.2, CON26.5, CON26.7, CON26.9
- new net AGND: C21.2, C22.2, C23.2, CON26.5, CON26.7, CON26.9
Changed lines of the file:
@@
 $EndDescr
 $Comp
-L GND #PWR060
+L GND #PWR053
 U 1 1 53943822
 P 1400 3250
-F 0 "#PWR060" H 1400 3250 30  0001 C CNN
+F 0 "#PWR053" H 1400 3250 30  0001 C CNN
 F 1 "GND" H 1400 3180 30  0001 C CNN
 F 2 "" H 1400 3250 60  0000 C CNN
@@
 Littelfuse MINI Blade Fuse\nmodel 0297015 (15A)\n% of rating | opening time max\n135%       | 600s\n200%       | 5 s \n350%       | 0.25 s \n600%       | 0.1 s\nReverse protection diode should \nwithstand at least 50A for 0.3s.
 $Comp
-L GND #PWR061
+L GND #PWR054
 U 1 1 53943829
 P 2900 3250
-F 0 "#PWR061" H 2900 3250 30  0001 C CNN
+F 0 "#PWR054" H 2900 3250 30  0001 C CNN
 F 1 "GND" H 2900 3180 30  0001 C CNN
 F 2 "" H 2900 3250 60  0000 C CNN
@@
 $EndComp
 $Comp
-L GND #PWR062
+L GND #PWR055
 U 1 1 5394382F
 P 2900 2550
-F 0 "#PWR062" H 2900 2550 30  0001 C CNN
+F 0 "#PWR055" H 2900 2550 30  0001 C CNN
 F 1 "GND" H 2900 2480 30  0001 C CNN
 F 2 "" H 2900 2550 60  0000 C CNN
@@
 $EndComp
 $Comp
-L GND #PWR063
+L GND #PWR056
 U 1 1 53943835
 P 2900 3950
-F 0 "#PWR063" H 2900 3950 30  0001 C CNN
+F 0 "#PWR056" H 2900 3950 30  0001 C CNN
 F 1 "GND" H 2900 3880 30  0001 C CNN
 F 2 "" H 2900 3950 60  0000 C CNN
@@
 $EndComp
 $Comp
-L GND #PWR064
+L GND #PWR057
 U 1 1 53943842
 P 1850 2550
-F 0 "#PWR064" H 1850 2550 30  0001 C CNN
+F 0 "#PWR057" H 1850 2550 30  0001 C CNN
 F 1 "GND" H 1850 2480 30  0001 C CNN
 F 2 "" H 1850 2550 60  0000 C CNN
@@
 $EndComp
 $Comp
-L GND #PWR065
+L GND #PWR058
 U 1 1 53943848
 P 1850 3250
-F 0 "#PWR065" H 1850 3250 30  0001 C CNN
+F 0 "#PWR058" H 1850 3250 30  0001 C CNN
 F 1 "GND" H 1850 3180 30  0001 C CNN
 F 2 "" H 1850 3250 60  0000 C CNN
@@
 $EndComp
 $Comp
-L GND #PWR066
+L GND #PWR059
 U 1 1 5394384E
 P 1850 3950
-F 0 "#PWR066" H 1850 3950 30  0001 C CNN
+F 0 "#PWR059" H 1850 3950 30  0001 C CNN
 F 1 "GND" H 1850 3880 30  0001 C CNN
 F 2 "" H 1850 3950 60  0000 C CNN
@@
 $EndComp
 $Comp
-L PWR_FLAG #FLG067
+L PWR_FLAG #FLG060
 U 1 1 539438AC
 P 3400 2050
-F 0 "#FLG067" H 3400 2145 30  0001 C CNN
+F 0 "#FLG060" H 3400 2145 30  0001 C CNN
 F 1 "PWR_FLAG" H 3400 2230 30  0000 C CNN
 F 2 "" H 3400 2050 60  0000 C CNN
@@
 $EndComp
 $Comp
-L PWR_FLAG #FLG068
+L PWR_FLAG #FLG061
 U 1 1 539438B2
 P 3400 2750
-F 0 "#FLG068" H 3400 2845 30  0001 C CNN
+F 0 "#FLG061" H 3400 2845 30  0001 C CNN
 F 1 "PWR_FLAG" H 3400 2930 30  0000 C CNN
 F 2 "" H 3400 2750 60  0000 C CNN
@@
 $EndComp
 $Comp
-L PWR_FLAG #FLG069
+L PWR_FLAG #FLG062
 U 1 1 539438B8
 P 3400 3450
-F 0 "#FLG069" H 3400 3545 30  0001 C CNN
+F 0 "#FLG062" H 3400 3545 30  0001 C CNN
 F 1 "PWR_FLAG" H 3400 3630 30  0000 C CNN
 F 2 "" H 3400 3450 60  0000 C CNN
@@
 $EndComp
 $Comp
-L PWR_FLAG #FLG070
+L PWR_FLAG #FLG063
 U 1 1 539438BE
 P 3400 4200
-F 0 "#FLG070" H 3400 4295 30  0001 C CNN
+F 0 "#FLG063" H 3400 4295 30  0001 C CNN
 F 1 "PWR_FLAG" H 3400 4380 30  0000 C CNN
 F 2 "" H 3400 4200 60  0000 C CNN
@@
 $EndComp
 $Comp
-L PWR_FLAG #FLG071
+L PWR_FLAG #FLG064
 U 1 1 539438C4
 P 1250 4750
-F 0 "#FLG071" H 1250 4845 30  0001 C CNN
+F 0 "#FLG064" H 1250 4845 30  0001 C CNN
 F 1 "PWR_FLAG" H 1250 4930 30  0000 C CNN
 F 2 "" H 1250 4750 60  0000 C CNN
@@
 $EndComp
 $Comp
-L GND #PWR072
+L GND #PWR065
 U 1 1 539438CA
 P 1250 4850
-F 0 "#PWR072" H 1250 4850 30  0001 C CNN
+F 0 "#PWR065" H 1250 4850 30  0001 C CNN
 F 1 "GND" H 1250 4780 30  0001 C CNN
 F 2 "" H 1250 4850 60  0000 C CNN
@@
 IOREF
 $Comp
-L PWR_FLAG #FLG073
+L PWR_FLAG #FLG066
 U 1 1 53943908
 P 1400 4150
-F 0 "#FLG073" H 1400 4245 30  0001 C CNN
+F 0 "#FLG066" H 1400 4245 30  0001 C CNN
 F 1 "PWR_FLAG" H 1400 4330 30  0000 C CNN
 F 2 "" H 1400 4150 60  0000 C CNN
@@
 $EndComp
 $Comp
-L PWR_FLAG #FLG074
+L PWR_FLAG #FLG067
 U 1 1 5394390F
 P 1100 4150
-F 0 "#FLG074" H 1100 4245 30  0001 C CNN
+F 0 "#FLG067" H 1100 4245 30  0001 C CNN
 F 1 "PWR_FLAG" H 1100 4330 30  0000 C CNN
 F 2 "" H 1100 4150 60  0000 C CNN
@@
 $EndComp
 $Comp
-L GND #PWR075
+L GND #PWR068
 U 1 1 53943ED6
 P 4850 4150
-F 0 "#PWR075" H 4850 4150 30  0001 C CNN
+F 0 "#PWR068" H 4850 4150 30  0001 C CNN
 F 1 "GND" H 4850 4080 30  0001 C CNN
 F 2 "" H 4850 4150 60  0000 C CNN
@@
 $EndComp
 $Comp
-L GND #PWR076
+L GND #PWR069
 U 1 1 53943F43
 P 4850 2900
-F 0 "#PWR076" H 4850 2900 30  0001 C CNN
+F 0 "#PWR069" H 4850 2900 30  0001 C CNN
 F 1 "GND" H 4850 2830 30  0001 C CNN
 F 2 "" H 4850 2900 60  0000 C CNN
@@
 D47
 $Comp
-L GND #PWR077
+L GND #PWR070
 U 1 1 53948CCE
 P 4150 6350
-F 0 "#PWR077" H 4150 6350 30  0001 C CNN
+F 0 "#PWR070" H 4150 6350 30  0001 C CNN
 F 1 "GND" H 4150 6280 30  0001 C CNN
 F 2 "" H 4150 6350 60  0000 C CNN
@@
 Connection ~ 3900 7150
 $Comp
-L GND #PWR078
+L GND #PWR071
 U 1 1 53949810
 P 3900 7200
-F 0 "#PWR078" H 3900 7200 30  0001 C CNN
+F 0 "#PWR071" H 3900 7200 30  0001 C CNN
 F 1 "GND" H 3900 7130 30  0001 C CNN
 F 2 "" H 3900 7200 60  0000 C CNN
@@
 $EndComp
 $Comp
-L GND #PWR079
+L GND #PWR072
 U 1 1 5394A1DE
 P 7550 3050
-F 0 "#PWR079" H 7550 3050 30  0001 C CNN
+F 0 "#PWR072" H 7550 3050 30  0001 C CNN
 F 1 "GND" H 7550 2980 30  0001 C CNN
 F 2 "" H 7550 3050 60  0000 C CNN
@@
 $EndComp
 $Comp
-L GND #PWR080
+L GND #PWR073
 U 1 1 5394A1E4
 P 7550 1800
-F 0 "#PWR080" H 7550 1800 30  0001 C CNN
+F 0 "#PWR073" H 7550 1800 30  0001 C CNN
 F 1 "GND" H 7550 1730 30  0001 C CNN
 F 2 "" H 7550 1800 60  0000 C CNN
@@
 	8600 1550 8500 1550
 Connection ~ 8500 1550
-$Comp
-L GND #PWR081
-U 1 1 5394B08E
-P 8500 1800
-F 0 "#PWR081" H 8500 1800 30  0001 C CNN
-F 1 "GND" H 8500 1730 30  0001 C CNN
-F 2 "" H 8500 1800 60  0000 C CNN
-F 3 "" H 8500 1800 60  0000 C CNN
-	1    8500 1800
-	1    0    0    -1
-$EndComp
 Wire Wire Line
 	9000 1450 9600 1450
@@
 	1    0    0    -1
 $EndComp
-$Comp
-L GND #PWR082
-U 1 1 5394B617
-P 7200 4450
-F 0 "#PWR082" H 7200 4450 30  0001 C CNN
-F 1 "GND" H 7200 4380 30  0001 C CNN
-F 2 "~" H 7200 4450 60  0000 C CNN
-F 3 "~" H 7200 4450 60  0000 C CNN
-	1    7200 4450
-	1    0    0    -1
-$EndComp
 Text GLabel 7100 3950 0    50   Input ~ 0
 A11
@@
 	1    0    0    -1
 $EndComp
-$Comp
-L GND #PWR083
-U 1 1 5394B93D
-P 9050 4450
-F 0 "#PWR083" H 9050 4450 30  0001 C CNN
-F 1 "GND" H 9050 4380 30  0001 C CNN
-F 2 "~" H 9050 4450 60  0000 C CNN
-F 3 "~" H 9050 4450 60  0000 C CNN
-	1    9050 4450
-	1    0    0    -1
-$EndComp
 Text GLabel 8950 3950 0    50   Input ~ 0
 A13
@@
 F 3 "~" H 9050 2950 60  0000 C CNN
 	1    9050 2950
-	1    0    0    -1
-$EndComp
-$Comp
-L GND #PWR084
-U 1 1 5394BA08
-P 9050 3200
-F 0 "#PWR084" H 9050 3200 30  0001 C CNN
-F 1 "GND" H 9050 3130 30  0001 C CNN
-F 2 "~" H 9050 3200 60  0000 C CNN
-F 3 "~" H 9050 3200 60  0000 C CNN
-	1    9050 3200
 	1    0    0    -1
 $EndComp
@@
 $EndComp
 $Comp
-L GND #PWR085
+L GND #PWR074
 U 1 1 539CFAEC
 P 3850 5850
-F 0 "#PWR085" H 3850 5850 30  0001 C CNN
+F 0 "#PWR074" H 3850 5850 30  0001 C CNN
 F 1 "GND" H 3850 5780 30  0001 C CNN
 F 2 "" H 3850 5850 60  0000 C CNN
@@
 $EndComp
 $Comp
-L GND #PWR086
+L GND #PWR075
 U 1 1 539CFEC7
 P 4500 3600
-F 0 "#PWR086" H 4500 3600 30  0001 C CNN
+F 0 "#PWR075" H 4500 3600 30  0001 C CNN
 F 1 "GND" H 4500 3530 30  0001 C CNN
 F 2 "" H 4500 3600 60  0000 C CNN
@@
 Connection ~ 7250 800
 $Comp
-L GND #PWR087
+L GND #PWR076
 U 1 1 539D0988
 P 7250 1250
-F 0 "#PWR087" H 7250 1250 30  0001 C CNN
+F 0 "#PWR076" H 7250 1250 30  0001 C CNN
 F 1 "GND" H 7250 1180 30  0001 C CNN
 F 2 "" H 7250 1250 60  0000 C CNN
@@
 	2650 4250 2650 2800
 Connection ~ 2650 2800
+Text GLabel 8500 1800 3    60   UnSpc ~ 0
+AGND
+Text GLabel 9050 3200 3    60   UnSpc ~ 0
+AGND
+Text GLabel 9050 4450 3    60   UnSpc ~ 0
+AGND
+Text GLabel 7200 4450 3    60   UnSpc ~ 0
+AGND
 $EndSCHEMATC
