File: kicad/power.sch (KiCad schematic (older format))
At the start: 32 parts, among them CON23 PS-ON, CON24 CON6, CON25 FAN, CON26 Chamber, Q7 FDC6401N, Q8 FDC6401N, Q9 FDC6401N

Commit message: Organize silkscreen.
Parts:
- F1: value MINI_Blade_Fuse_Holder -> BED
- F2: value MINI_Blade_Fuse_Holder -> Heaters
- F3: value MINI_Blade_Fuse_Holder -> Motors
Changed lines of the file:
@@
 P 2400 2100
 F 0 "F1" H 2400 2240 60  0000 C CNN
-F 1 "MINI_Blade_Fuse_Holder" H 2400 2015 60  0001 C CNN
+F 1 "BED" H 2400 2015 60  0000 C CNN
 F 2 "Littlefuse_01530008" H 2390 2170 40  0000 C CNN
 F 3 "" V 2400 2100 30  0000 C CNN
@@
 P 2300 2800
 F 0 "F2" H 2300 2940 60  0000 C CNN
-F 1 "MINI_Blade_Fuse_Holder" H 2300 2715 60  0001 C CNN
+F 1 "Heaters" H 2300 2715 60  0000 C CNN
 F 2 "Littlefuse_01530008" H 2290 2870 40  0000 C CNN
 F 3 "" V 2300 2800 30  0000 C CNN
@@
 P 2300 3500
 F 0 "F3" H 2300 3640 60  0000 C CNN
-F 1 "MINI_Blade_Fuse_Holder" H 2300 3415 60  0001 C CNN
+F 1 "Motors" H 2300 3415 60  0000 C CNN
 F 2 "Littlefuse_01530008" H 2290 3570 40  0000 C CNN
 F 3 "" V 2300 3500 30  0000 C CNN
