File: kicad/YZaxis.sch (KiCad schematic (older format))
At the start: 38 parts, among them CON16 YZ, CON17 Stepstick_Left_Connector, CON18 Stepstick_Right_Connector, CON19 Stepstick_Left_Connector, CON20 Stepstick_Right_Connector, CON27 BED, CON28 BED_Th, Q5 IRLR2905ZPBF, Q6 FDC6401N, U1 CD4504BPW

Commit message: Place
Parts:
- removed CON16: YZ, IDC34, symbol CON17x2
- added C26: 100n/50V, 0603, symbol C
- added CON16: CON14x2, IDC28, symbol CON14x2
- gave numbers to parts that had none: 2
Connections:
- net +12V: now also C26.1, CON16.26, CON16.28
- net +5V: now also CON16.13, CON16.16, CON16.5, CON16.8
- net GND: now also C26.2, CON16.12, CON16.15, CON16.6, CON16.9
- net OC5: now also CON16.25
- net OC6: now also CON16.27
- net Ymax: now also CON16.14
- net Ymin: now also CON16.7
- net YmotorA: now also CON16.1
- net YmotorB: now also CON16.2
- net YmotorC: now also CON16.3
- net YmotorD: now also CON16.4
- net Zmax: now also CON16.10
- net Zmin: now also CON16.11
- net ZmotorA: now also CON16.17, CON16.21
- net ZmotorB: now also CON16.18, CON16.22
- net ZmotorC: now also CON16.19, CON16.23
- net ZmotorD: now also CON16.20, CON16.24
- no-connect marks 9 -> 3
Changed lines of the file:
@@
 A7
 $Comp
-L GND #PWR027
+L GND #PWR49
 U 1 1 534EC7A3
 P 2550 7250
-F 0 "#PWR027" H 2550 7250 30  0001 C CNN
+F 0 "#PWR49" H 2550 7250 30  0001 C CNN
 F 1 "GND" H 2550 7180 30  0001 C CNN
 F 2 "~" H 2550 7250 60  0000 C CNN
@@
 $EndComp
 $Comp
-L GND #PWR028
+L GND #PWR50
 U 1 1 534ECB96
 P 4500 7400
-F 0 "#PWR028" H 4500 7400 30  0001 C CNN
+F 0 "#PWR50" H 4500 7400 30  0001 C CNN
 F 1 "GND" H 4500 7330 30  0001 C CNN
 F 2 "~" H 4500 7400 60  0000 C CNN
@@
 Connection ~ 4500 6850
 $Comp
-L GND #PWR029
+L GND #PWR34
 U 1 1 534ED3BB
 P 9900 2250
-F 0 "#PWR029" H 9900 2250 30  0001 C CNN
+F 0 "#PWR34" H 9900 2250 30  0001 C CNN
 F 1 "GND" H 9900 2180 30  0001 C CNN
 F 2 "~" H 9900 2250 60  0000 C CNN
@@
 $EndComp
 $Comp
-L GND #PWR030
+L GND #PWR35
 U 1 1 534ED3D4
 P 10300 2250
-F 0 "#PWR030" H 10300 2250 30  0001 C CNN
+F 0 "#PWR35" H 10300 2250 30  0001 C CNN
 F 1 "GND" H 10300 2180 30  0001 C CNN
 F 2 "~" H 10300 2250 60  0000 C CNN
@@
 $EndComp
 $Comp
-L GND #PWR031
+L GND #PWR32
 U 1 1 534ED3DA
 P 9100 2250
-F 0 "#PWR031" H 9100 2250 30  0001 C CNN
+F 0 "#PWR32" H 9100 2250 30  0001 C CNN
 F 1 "GND" H 9100 2180 30  0001 C CNN
 F 2 "~" H 9100 2250 60  0000 C CNN
@@
 	1000 7100 1300 7100
 $Comp
-L GND #PWR032
+L GND #PWR52
 U 1 1 536FED2A
 P 1150 7500
-F 0 "#PWR032" H 1150 7500 30  0001 C CNN
+F 0 "#PWR52" H 1150 7500 30  0001 C CNN
 F 1 "GND" H 1150 7430 30  0001 C CNN
 F 2 "~" H 1150 7500 60  0000 C CNN
@@
 	7850 5300 7850 5400
 $Comp
-L GND #PWR033
+L GND #PWR45
 U 1 1 537E6A4E
 P 7850 5400
-F 0 "#PWR033" H 7850 5400 30  0001 C CNN
+F 0 "#PWR45" H 7850 5400 30  0001 C CNN
 F 1 "GND" H 7850 5330 30  0001 C CNN
 F 2 "~" H 7850 5400 60  0000 C CNN
@@
 	7850 6100 7850 6200
 $Comp
-L GND #PWR034
+L GND #PWR47
 U 1 1 537E6A65
 P 7850 6200
-F 0 "#PWR034" H 7850 6200 30  0001 C CNN
+F 0 "#PWR47" H 7850 6200 30  0001 C CNN
 F 1 "GND" H 7850 6130 30  0001 C CNN
 F 2 "~" H 7850 6200 60  0000 C CNN
@@
 	9500 5350 9500 5450
 $Comp
-L GND #PWR035
+L GND #PWR46
 U 1 1 537E6A80
 P 9500 5450
-F 0 "#PWR035" H 9500 5450 30  0001 C CNN
+F 0 "#PWR46" H 9500 5450 30  0001 C CNN
 F 1 "GND" H 9500 5380 30  0001 C CNN
 F 2 "~" H 9500 5450 60  0000 C CNN
@@
 	9500 6150 9500 6250
 $Comp
-L GND #PWR036
+L GND #PWR48
 U 1 1 537E6A97
 P 9500 6250
-F 0 "#PWR036" H 9500 6250 30  0001 C CNN
+F 0 "#PWR48" H 9500 6250 30  0001 C CNN
 F 1 "GND" H 9500 6180 30  0001 C CNN
 F 2 "~" H 9500 6250 60  0000 C CNN
@@
 	6400 1800 5850 1800
 $Comp
-L GND #PWR037
+L GND #PWR29
 U 1 1 537E6E27
 P 6650 1500
-F 0 "#PWR037" H 6650 1500 30  0001 C CNN
+F 0 "#PWR29" H 6650 1500 30  0001 C CNN
 F 1 "GND" H 6650 1430 30  0001 C CNN
 F 2 "~" H 6650 1500 60  0000 C CNN
@@
 	4750 1000 4750 1500
 $Comp
-L GND #PWR038
+L GND #PWR30
 U 1 1 537E72EF
 P 4650 1700
-F 0 "#PWR038" H 4650 1700 30  0001 C CNN
+F 0 "#PWR30" H 4650 1700 30  0001 C CNN
 F 1 "GND" H 4650 1630 30  0001 C CNN
 F 2 "~" H 4650 1700 60  0000 C CNN
@@
 Wire Wire Line
 	4900 2200 5450 2200
-$Comp
-L CON17x2 CON16
-U 1 1 537E808F
-P 5650 1700
-F 0 "CON16" H 5650 2620 60  0000 C CNN
-F 1 "YZ" H 5650 800 60  0000 C CNN
-F 2 "IDC34" H 5650 700 40  0000 C CNN
-F 3 "" H 5650 1700 40  0000 C CNN
-	1    5650 1700
-	1    0    0    -1
-$EndComp
 NoConn ~ 8400 1900
 Text GLabel 6550 1000 1    60   UnSpc ~ 0
@@
 Text GLabel 4750 1000 1    60   UnSpc ~ 0
 +5V
-NoConn ~ 5450 2300
-NoConn ~ 5450 2400
-NoConn ~ 5450 2500
-NoConn ~ 5850 2500
-NoConn ~ 5850 2400
-NoConn ~ 5850 2300
 Wire Wire Line
 	9500 1450 9500 1600
@@
 Connection ~ 7800 1450
 $Comp
-L GND #PWR039
+L GND #PWR31
 U 1 1 538D7812
 P 7800 2150
-F 0 "#PWR039" H 7800 2150 30  0001 C CNN
+F 0 "#PWR31" H 7800 2150 30  0001 C CNN
 F 1 "GND" H 7800 2080 30  0001 C CNN
 F 2 "~" H 7800 2150 60  0000 C CNN
@@
 $EndComp
 $Comp
-L GND #PWR040
+L GND #PWR33
 U 1 1 538D791A
 P 9500 2250
-F 0 "#PWR040" H 9500 2250 30  0001 C CNN
+F 0 "#PWR33" H 9500 2250 30  0001 C CNN
 F 1 "GND" H 9500 2180 30  0001 C CNN
 F 2 "~" H 9500 2250 60  0000 C CNN
@@
 $EndComp
 $Comp
-L GND #PWR041
+L GND #PWR40
 U 1 1 53924614
 P 8150 4000
-F 0 "#PWR041" H 8150 4000 30  0001 C CNN
+F 0 "#PWR40" H 8150 4000 30  0001 C CNN
 F 1 "GND" H 8150 3930 30  0001 C CNN
 F 2 "~" H 8150 4000 60  0000 C CNN
@@
 	8150 4000 8150 3950
 $Comp
-L GND #PWR042
+L GND #PWR41
 U 1 1 5392461B
 P 9450 4000
-F 0 "#PWR042" H 9450 4000 30  0001 C CNN
+F 0 "#PWR41" H 9450 4000 30  0001 C CNN
 F 1 "GND" H 9450 3930 30  0001 C CNN
 F 2 "~" H 9450 4000 60  0000 C CNN
@@
 +12V
 Wire Wire Line
-	8250 2950 8150 2950
+	7750 2950 8250 2950
 Wire Wire Line
 	8150 2950 8150 3050
@@
 $EndComp
 $Comp
-L GND #PWR043
+L GND #PWR38
 U 1 1 539A1B02
 P 3200 2900
-F 0 "#PWR043" H 3200 2900 30  0001 C CNN
+F 0 "#PWR38" H 3200 2900 30  0001 C CNN
 F 1 "GND" H 3200 2830 30  0001 C CNN
 F 2 "~" H 3200 2900 60  0000 C CNN
@@
 Z
 $Comp
-L GND #PWR044
+L GND #PWR36
 U 1 1 539A1B17
 P 2000 2900
-F 0 "#PWR044" H 2000 2900 30  0001 C CNN
+F 0 "#PWR36" H 2000 2900 30  0001 C CNN
 F 1 "GND" H 2000 2830 30  0001 C CNN
 F 2 "~" H 2000 2900 60  0000 C CNN
@@
 $EndComp
 $Comp
-L GND #PWR045
+L GND #PWR37
 U 1 1 539A1B1D
 P 3000 2900
-F 0 "#PWR045" H 3000 2900 30  0001 C CNN
+F 0 "#PWR37" H 3000 2900 30  0001 C CNN
 F 1 "GND" H 3000 2830 30  0001 C CNN
 F 2 "~" H 3000 2900 60  0000 C CNN
@@
 $EndComp
 $Comp
-L GND #PWR046
+L GND #PWR44
 U 1 1 539A1C4E
 P 3200 5250
-F 0 "#PWR046" H 3200 5250 30  0001 C CNN
+F 0 "#PWR44" H 3200 5250 30  0001 C CNN
 F 1 "GND" H 3200 5180 30  0001 C CNN
 F 2 "~" H 3200 5250 60  0000 C CNN
@@
 Y
 $Comp
-L GND #PWR047
+L GND #PWR42
 U 1 1 539A1C63
 P 2000 5250
-F 0 "#PWR047" H 2000 5250 30  0001 C CNN
+F 0 "#PWR42" H 2000 5250 30  0001 C CNN
 F 1 "GND" H 2000 5180 30  0001 C CNN
 F 2 "~" H 2000 5250 60  0000 C CNN
@@
 $EndComp
 $Comp
-L GND #PWR048
+L GND #PWR43
 U 1 1 539A1C69
 P 3000 5250
-F 0 "#PWR048" H 3000 5250 30  0001 C CNN
+F 0 "#PWR43" H 3000 5250 30  0001 C CNN
 F 1 "GND" H 3000 5180 30  0001 C CNN
 F 2 "~" H 3000 5250 60  0000 C CNN
@@
 	5100 6950 5100 7400
 $Comp
-L GND #PWR049
+L GND #PWR51
 U 1 1 539C8F1D
 P 5100 7400
-F 0 "#PWR049" H 5100 7400 30  0001 C CNN
+F 0 "#PWR51" H 5100 7400 30  0001 C CNN
 F 1 "GND" H 5100 7330 30  0001 C CNN
 F 2 "~" H 5100 7400 60  0000 C CNN
@@
 Connection ~ 4500 6900
 $Comp
-L PMEG3010EJ D?
+L PMEG3010EJ D13
 U 1 1 539CCE24
 P 8150 3200
-F 0 "D?" H 8150 3400 60  0000 C CNN
-F 1 "PMEG3010EJ" H 8150 3300 60  0000 C CNN
+F 0 "D13" H 8150 3400 60  0000 C CNN
+F 1 "PMEG3010EJ" H 8100 3300 60  0000 C CNN
 F 2 "SOD323F" H 8150 3100 30  0000 C CNN
 F 3 "" V 8150 3200 60  0000 C CNN
@@
 $EndComp
 $Comp
-L PMEG3010EJ D?
+L PMEG3010EJ D14
 U 1 1 539CD76F
 P 9450 3200
-F 0 "D?" H 9450 3400 60  0000 C CNN
+F 0 "D14" H 9450 3400 60  0000 C CNN
 F 1 "PMEG3010EJ" H 9450 3300 60  0000 C CNN
 F 2 "SOD323F" H 9450 3100 30  0000 C CNN
@@
 	0    -1   -1   0
 $EndComp
+$Comp
+L C C26
+U 1 1 539D1A87
+P 7750 3200
+F 0 "C26" H 7755 3285 60  0000 L CNN
+F 1 "100n/50V" H 7756 3115 60  0000 L CNN
+F 2 "0603" H 7850 3050 30  0000 C CNN
+F 3 "~" H 7750 3200 60  0000 C CNN
+	1    7750 3200
+	-1   0    0    -1
+$EndComp
+Wire Wire Line
+	7750 2950 7750 3050
+Connection ~ 8150 2950
+Wire Wire Line
+	7750 3350 7750 3400
+$Comp
+L GND #PWR39
+U 1 1 539D1ECC
+P 7750 3400
+F 0 "#PWR39" H 7750 3400 30  0001 C CNN
+F 1 "GND" H 7750 3330 30  0001 C CNN
+F 2 "~" H 7750 3400 60  0000 C CNN
+F 3 "~" H 7750 3400 60  0000 C CNN
+	1    7750 3400
+	1    0    0    -1
+$EndComp
+$Comp
+L CON14x2 CON16
+U 1 1 539D4BA5
+P 5650 1550
+F 0 "CON16" H 5650 2320 60  0000 C CNN
+F 1 "CON14x2" H 5650 800 60  0000 C CNN
+F 2 "IDC28" H 5650 1550 40  0000 C CNN
+F 3 "" H 5650 1550 40  0000 C CNN
+	1    5650 1550
+	1    0    0    -1
+$EndComp
 $EndSCHEMATC

Commit message: Fix panel connections. Place.
Parts:
- CON16: footprint IDC28 -> YZ
Changed lines of the file:
@@
 A7
 $Comp
-L GND #PWR49
+L GND #PWR029
 U 1 1 534EC7A3
 P 2550 7250
-F 0 "#PWR49" H 2550 7250 30  0001 C CNN
+F 0 "#PWR029" H 2550 7250 30  0001 C CNN
 F 1 "GND" H 2550 7180 30  0001 C CNN
 F 2 "~" H 2550 7250 60  0000 C CNN
@@
 $EndComp
 $Comp
-L GND #PWR50
+L GND #PWR030
 U 1 1 534ECB96
 P 4500 7400
-F 0 "#PWR50" H 4500 7400 30  0001 C CNN
+F 0 "#PWR030" H 4500 7400 30  0001 C CNN
 F 1 "GND" H 4500 7330 30  0001 C CNN
 F 2 "~" H 4500 7400 60  0000 C CNN
@@
 Connection ~ 4500 6850
 $Comp
-L GND #PWR34
+L GND #PWR031
 U 1 1 534ED3BB
 P 9900 2250
-F 0 "#PWR34" H 9900 2250 30  0001 C CNN
+F 0 "#PWR031" H 9900 2250 30  0001 C CNN
 F 1 "GND" H 9900 2180 30  0001 C CNN
 F 2 "~" H 9900 2250 60  0000 C CNN
@@
 $EndComp
 $Comp
-L GND #PWR35
+L GND #PWR032
 U 1 1 534ED3D4
 P 10300 2250
-F 0 "#PWR35" H 10300 2250 30  0001 C CNN
+F 0 "#PWR032" H 10300 2250 30  0001 C CNN
 F 1 "GND" H 10300 2180 30  0001 C CNN
 F 2 "~" H 10300 2250 60  0000 C CNN
@@
 $EndComp
 $Comp
-L GND #PWR32
+L GND #PWR033
 U 1 1 534ED3DA
 P 9100 2250
-F 0 "#PWR32" H 9100 2250 30  0001 C CNN
+F 0 "#PWR033" H 9100 2250 30  0001 C CNN
 F 1 "GND" H 9100 2180 30  0001 C CNN
 F 2 "~" H 9100 2250 60  0000 C CNN
@@
 	1000 7100 1300 7100
 $Comp
-L GND #PWR52
+L GND #PWR034
 U 1 1 536FED2A
 P 1150 7500
-F 0 "#PWR52" H 1150 7500 30  0001 C CNN
+F 0 "#PWR034" H 1150 7500 30  0001 C CNN
 F 1 "GND" H 1150 7430 30  0001 C CNN
 F 2 "~" H 1150 7500 60  0000 C CNN
@@
 	7850 5300 7850 5400
 $Comp
-L GND #PWR45
+L GND #PWR035
 U 1 1 537E6A4E
 P 7850 5400
-F 0 "#PWR45" H 7850 5400 30  0001 C CNN
+F 0 "#PWR035" H 7850 5400 30  0001 C CNN
 F 1 "GND" H 7850 5330 30  0001 C CNN
 F 2 "~" H 7850 5400 60  0000 C CNN
@@
 	7850 6100 7850 6200
 $Comp
-L GND #PWR47
+L GND #PWR036
 U 1 1 537E6A65
 P 7850 6200
-F 0 "#PWR47" H 7850 6200 30  0001 C CNN
+F 0 "#PWR036" H 7850 6200 30  0001 C CNN
 F 1 "GND" H 7850 6130 30  0001 C CNN
 F 2 "~" H 7850 6200 60  0000 C CNN
@@
 	9500 5350 9500 5450
 $Comp
-L GND #PWR46
+L GND #PWR037
 U 1 1 537E6A80
 P 9500 5450
-F 0 "#PWR46" H 9500 5450 30  0001 C CNN
+F 0 "#PWR037" H 9500 5450 30  0001 C CNN
 F 1 "GND" H 9500 5380 30  0001 C CNN
 F 2 "~" H 9500 5450 60  0000 C CNN
@@
 	9500 6150 9500 6250
 $Comp
-L GND #PWR48
+L GND #PWR038
 U 1 1 537E6A97
 P 9500 6250
-F 0 "#PWR48" H 9500 6250 30  0001 C CNN
+F 0 "#PWR038" H 9500 6250 30  0001 C CNN
 F 1 "GND" H 9500 6180 30  0001 C CNN
 F 2 "~" H 9500 6250 60  0000 C CNN
@@
 	6400 1800 5850 1800
 $Comp
-L GND #PWR29
+L GND #PWR039
 U 1 1 537E6E27
 P 6650 1500
-F 0 "#PWR29" H 6650 1500 30  0001 C CNN
+F 0 "#PWR039" H 6650 1500 30  0001 C CNN
 F 1 "GND" H 6650 1430 30  0001 C CNN
 F 2 "~" H 6650 1500 60  0000 C CNN
@@
 	4750 1000 4750 1500
 $Comp
-L GND #PWR30
+L GND #PWR040
 U 1 1 537E72EF
 P 4650 1700
-F 0 "#PWR30" H 4650 1700 30  0001 C CNN
+F 0 "#PWR040" H 4650 1700 30  0001 C CNN
 F 1 "GND" H 4650 1630 30  0001 C CNN
 F 2 "~" H 4650 1700 60  0000 C CNN
@@
 Connection ~ 7800 1450
 $Comp
-L GND #PWR31
+L GND #PWR041
 U 1 1 538D7812
 P 7800 2150
-F 0 "#PWR31" H 7800 2150 30  0001 C CNN
+F 0 "#PWR041" H 7800 2150 30  0001 C CNN
 F 1 "GND" H 7800 2080 30  0001 C CNN
 F 2 "~" H 7800 2150 60  0000 C CNN
@@
 $EndComp
 $Comp
-L GND #PWR33
+L GND #PWR042
 U 1 1 538D791A
 P 9500 2250
-F 0 "#PWR33" H 9500 2250 30  0001 C CNN
+F 0 "#PWR042" H 9500 2250 30  0001 C CNN
 F 1 "GND" H 9500 2180 30  0001 C CNN
 F 2 "~" H 9500 2250 60  0000 C CNN
@@
 $EndComp
 $Comp
-L GND #PWR40
+L GND #PWR043
 U 1 1 53924614
 P 8150 4000
-F 0 "#PWR40" H 8150 4000 30  0001 C CNN
+F 0 "#PWR043" H 8150 4000 30  0001 C CNN
 F 1 "GND" H 8150 3930 30  0001 C CNN
 F 2 "~" H 8150 4000 60  0000 C CNN
@@
 	8150 4000 8150 3950
 $Comp
-L GND #PWR41
+L GND #PWR044
 U 1 1 5392461B
 P 9450 4000
-F 0 "#PWR41" H 9450 4000 30  0001 C CNN
+F 0 "#PWR044" H 9450 4000 30  0001 C CNN
 F 1 "GND" H 9450 3930 30  0001 C CNN
 F 2 "~" H 9450 4000 60  0000 C CNN
@@
 $EndComp
 $Comp
-L GND #PWR38
+L GND #PWR045
 U 1 1 539A1B02
 P 3200 2900
-F 0 "#PWR38" H 3200 2900 30  0001 C CNN
+F 0 "#PWR045" H 3200 2900 30  0001 C CNN
 F 1 "GND" H 3200 2830 30  0001 C CNN
 F 2 "~" H 3200 2900 60  0000 C CNN
@@
 Z
 $Comp
-L GND #PWR36
+L GND #PWR046
 U 1 1 539A1B17
 P 2000 2900
-F 0 "#PWR36" H 2000 2900 30  0001 C CNN
+F 0 "#PWR046" H 2000 2900 30  0001 C CNN
 F 1 "GND" H 2000 2830 30  0001 C CNN
 F 2 "~" H 2000 2900 60  0000 C CNN
@@
 $EndComp
 $Comp
-L GND #PWR37
+L GND #PWR047
 U 1 1 539A1B1D
 P 3000 2900
-F 0 "#PWR37" H 3000 2900 30  0001 C CNN
+F 0 "#PWR047" H 3000 2900 30  0001 C CNN
 F 1 "GND" H 3000 2830 30  0001 C CNN
 F 2 "~" H 3000 2900 60  0000 C CNN
@@
 $EndComp
 $Comp
-L GND #PWR44
+L GND #PWR048
 U 1 1 539A1C4E
 P 3200 5250
-F 0 "#PWR44" H 3200 5250 30  0001 C CNN
+F 0 "#PWR048" H 3200 5250 30  0001 C CNN
 F 1 "GND" H 3200 5180 30  0001 C CNN
 F 2 "~" H 3200 5250 60  0000 C CNN
@@
 Y
 $Comp
-L GND #PWR42
+L GND #PWR049
 U 1 1 539A1C63
 P 2000 5250
-F 0 "#PWR42" H 2000 5250 30  0001 C CNN
+F 0 "#PWR049" H 2000 5250 30  0001 C CNN
 F 1 "GND" H 2000 5180 30  0001 C CNN
 F 2 "~" H 2000 5250 60  0000 C CNN
@@
 $EndComp
 $Comp
-L GND #PWR43
+L GND #PWR050
 U 1 1 539A1C69
 P 3000 5250
-F 0 "#PWR43" H 3000 5250 30  0001 C CNN
+F 0 "#PWR050" H 3000 5250 30  0001 C CNN
 F 1 "GND" H 3000 5180 30  0001 C CNN
 F 2 "~" H 3000 5250 60  0000 C CNN
@@
 	5100 6950 5100 7400
 $Comp
-L GND #PWR51
+L GND #PWR051
 U 1 1 539C8F1D
 P 5100 7400
-F 0 "#PWR51" H 5100 7400 30  0001 C CNN
+F 0 "#PWR051" H 5100 7400 30  0001 C CNN
 F 1 "GND" H 5100 7330 30  0001 C CNN
 F 2 "~" H 5100 7400 60  0000 C CNN
@@
 	7750 3350 7750 3400
 $Comp
-L GND #PWR39
+L GND #PWR052
 U 1 1 539D1ECC
 P 7750 3400
-F 0 "#PWR39" H 7750 3400 30  0001 C CNN
+F 0 "#PWR052" H 7750 3400 30  0001 C CNN
 F 1 "GND" H 7750 3330 30  0001 C CNN
 F 2 "~" H 7750 3400 60  0000 C CNN
@@
 F 0 "CON16" H 5650 2320 60  0000 C CNN
 F 1 "CON14x2" H 5650 800 60  0000 C CNN
-F 2 "IDC28" H 5650 1550 40  0000 C CNN
+F 2 "YZ" H 5650 1550 40  0000 C CNN
 F 3 "" H 5650 1550 40  0000 C CNN
 	1    5650 1550

Commit message: Route.
Connections:
- net D44: now also Q6.3 (G); no longer Q6.1 (G)
- net D45: now also Q6.1 (G); no longer Q6.3 (G)
- net OC5: now also Q6.4 (D); no longer Q6.6 (D)
- net OC6: now also Q6.6 (D); no longer Q6.4 (D)
Other:
- moved on the sheet: Q6A, Q6B
Changed lines of the file:
@@
 L FDC6401N Q6
 U 1 1 53924606
+P 9350 3750
+F 0 "Q6" H 9530 3820 60  0000 L CNN
+F 1 "FDC6401N" H 9530 3740 60  0000 L CNN
+F 2 "SOT23-6" H 9530 3670 40  0000 L CNN
+F 3 "" H 9350 3700 60  0000 C CNN
+	1    9350 3750
+	1    0    0    -1
+$EndComp
+$Comp
+L FDC6401N Q6
+U 2 1 5392460D
 P 8050 3750
 F 0 "Q6" H 8230 3820 60  0000 L CNN
@@
 F 2 "SOT23-6" H 8230 3670 40  0000 L CNN
 F 3 "" H 8050 3700 60  0000 C CNN
-	1    8050 3750
+	2    8050 3750
 	1    0    0    -1
 $EndComp
-$Comp
-L FDC6401N Q6
-U 2 1 5392460D
-P 9350 3750
-F 0 "Q6" H 9530 3820 60  0000 L CNN
-F 1 "FDC6401N" H 9530 3740 60  0000 L CNN
-F 2 "SOT23-6" H 9530 3670 40  0000 L CNN
-F 3 "" H 9350 3700 60  0000 C CNN
-	2    9350 3750
-	1    0    0    -1
-$EndComp

Commit message: Swap pins
Connections:
- net A7 is gone; now on net A2: CON19.8 (DIR)
- net D18 is gone; now on net D14: C16.1, R25.1
- net D48 is gone; now on net A6: CON17.8 (DIR)
- net A2: no longer CON19.1 (~EN), R23.2
- net A6: no longer CON19.7 (STEP)
- net D14: no longer C15.1, R24.1
- net A8 renamed A4
- net D15 renamed D25
- net D19 renamed D3
- net D46 renamed A5
- new net A0: CON19.1 (~EN), R23.2
- new net A1: CON19.7 (STEP)
- new net D2: C15.1, R24.1
Changed lines of the file:
@@
 $EndDescr
 Text GLabel 1300 3950 0    50   Input ~ 0
+A0
+Text GLabel 1300 4650 0    50   Input ~ 0
+A1
+Text GLabel 1300 4750 0    50   Input ~ 0
 A2
-Text GLabel 1300 4650 0    50   Input ~ 0
-A6
-Text GLabel 1300 4750 0    50   Input ~ 0
-A7
 $Comp
 L GND #PWR029
@@
 $EndComp
 Text GLabel 1300 1600 0    50   Input ~ 0
-A8
+A4
 Text GLabel 1300 2300 0    50   Input ~ 0
-D46
+A5
 Text GLabel 1300 2400 0    50   Input ~ 0
-D48
+A6
 Text Label 3850 1900 2    60   ~ 0
 ZmotorA
@@
 Ymax
 Text GLabel 7750 4900 0    50   Input ~ 0
-D14
+D2
 Text GLabel 7750 5700 0    50   Input ~ 0
-D15
+D25
 $Comp
 L R R24
@@
 Zmax
 Text GLabel 9400 4950 0    50   Input ~ 0
-D18
+D14
 Text GLabel 9400 5750 0    50   Input ~ 0
-D19
+D3
 $Comp
 L R R25

Commit message: Exchange stepstick connections.
Simplify layout
Parts:
- removed C19: 100u/35V, Cpol-6.3x7.7, symbol Cpol
- removed CON19: Stepstick_Left_Connector, PIN8, symbol Stepstick_Left_Connector
- removed CON20: Stepstick_Right_Connector, PIN8, symbol Stepstick_Right_Connector
- removed JP5: Jumper3, PIN3x2, symbol Jumper3
- removed MECH6: Y, symbol stepstickFootprint
- removed R23, R28: 22k, 0603, symbol R
- added C10: 100u/35V, Cpol-6.3x7.7, symbol Cpol
- added CON14: Stepstick_Left_Connector, PIN8, symbol Stepstick_Left_Connector
- added CON15: Stepstick_Right_Connector, PIN8, symbol Stepstick_Right_Connector
- added JP3: Jumper3, PIN3x2, symbol Jumper3
- added MECH4: Z, symbol stepstickFootprint
- added R14, R16: 22k, 0603, symbol R
- MECH5: value Z -> Y
Connections:
- net GND: now also C10.2, CON15.2 (GND), CON15.8 (GND), R16.2
- net IOREF: now also CON15.7 (VDD), JP3.2, JP3.4, JP3.6, R14.1
- net Vmot: now also C10.1, CON15.1 (VMOT)
- net YmotorA: now also CON18.3 (2B)
- net YmotorB: now also CON18.4 (2A)
- net YmotorC: now also CON18.5 (1A)
- net YmotorD: now also CON18.6 (1B)
- net ZmotorA: now also CON15.3 (2B); no longer CON18.3 (2B)
- net ZmotorB: now also CON15.4 (2A); no longer CON18.4 (2A)
- net ZmotorC: now also CON15.5 (1A); no longer CON18.5 (1A)
- net ZmotorD: now also CON15.6 (1B); no longer CON18.6 (1B)
- new net: CON14.2 (MS1), JP3.1, R16.1
- new net: CON14.3 (MS2), JP3.3
- new net: CON14.4 (MS3), JP3.5
- new net: CON14.5 (~RST), CON14.6 (~SLP)
- new net D36: CON14.1 (~EN), R14.2
- new net D38: CON14.7 (STEP)
- new net D46: CON14.8 (DIR)
Other:
- moved on the sheet: C13, CON17, CON18, JP4, MECH5, R17, R19

Commit message: Pin swap. Route.
Connections:
- net A15 renamed A10
Changed lines of the file:
@@
 	4500 6750 4500 7000
 Text GLabel 4400 6900 0    50   Input ~ 0
-A15
+A10
 Connection ~ 4500 6850
 $Comp
