File: kicad/YZaxis.sch (KiCad schematic (older format))
At the start: 39 parts, among them CON14 Stepstick_Left_Connector, CON15 Stepstick_Right_Connector, CON16 CON14x2, CON17 Stepstick_Left_Connector, CON18 Stepstick_Right_Connector, CON27 BED, CON28 BED_Th, Q5 IRLR2905ZPBF, Q6 FDC6401N, U1 CD4504BPW

Commit message: Add AGND. Route.
close #27
Connections:
- net GND: no longer C14.2, CON28.2
- new net AGND: C14.2, CON28.2
Changed lines of the file:
@@
 $EndDescr
 $Comp
-L GND #PWR029
+L GND #PWR024
 U 1 1 534EC7A3
 P 2550 7250
-F 0 "#PWR029" H 2550 7250 30  0001 C CNN
+F 0 "#PWR024" H 2550 7250 30  0001 C CNN
 F 1 "GND" H 2550 7180 30  0001 C CNN
 F 2 "~" H 2550 7250 60  0000 C CNN
@@
 	1    0    0    -1
 $EndComp
-$Comp
-L GND #PWR030
-U 1 1 534ECB96
-P 4500 7400
-F 0 "#PWR030" H 4500 7400 30  0001 C CNN
-F 1 "GND" H 4500 7330 30  0001 C CNN
-F 2 "~" H 4500 7400 60  0000 C CNN
-F 3 "~" H 4500 7400 60  0000 C CNN
-	1    4500 7400
-	1    0    0    -1
-$EndComp
 Wire Wire Line
 	4500 7400 4500 7300
@@
 Connection ~ 4500 6850
 $Comp
-L GND #PWR031
+L GND #PWR025
 U 1 1 534ED3BB
 P 9900 2250
-F 0 "#PWR031" H 9900 2250 30  0001 C CNN
+F 0 "#PWR025" H 9900 2250 30  0001 C CNN
 F 1 "GND" H 9900 2180 30  0001 C CNN
 F 2 "~" H 9900 2250 60  0000 C CNN
@@
 $EndComp
 $Comp
-L GND #PWR032
+L GND #PWR026
 U 1 1 534ED3D4
 P 10300 2250
-F 0 "#PWR032" H 10300 2250 30  0001 C CNN
+F 0 "#PWR026" H 10300 2250 30  0001 C CNN
 F 1 "GND" H 10300 2180 30  0001 C CNN
 F 2 "~" H 10300 2250 60  0000 C CNN
@@
 $EndComp
 $Comp
-L GND #PWR033
+L GND #PWR027
 U 1 1 534ED3DA
 P 9100 2250
-F 0 "#PWR033" H 9100 2250 30  0001 C CNN
+F 0 "#PWR027" H 9100 2250 30  0001 C CNN
 F 1 "GND" H 9100 2180 30  0001 C CNN
 F 2 "~" H 9100 2250 60  0000 C CNN
@@
 	1000 7100 1300 7100
 $Comp
-L GND #PWR034
+L GND #PWR028
 U 1 1 536FED2A
 P 1150 7500
-F 0 "#PWR034" H 1150 7500 30  0001 C CNN
+F 0 "#PWR028" H 1150 7500 30  0001 C CNN
 F 1 "GND" H 1150 7430 30  0001 C CNN
 F 2 "~" H 1150 7500 60  0000 C CNN
@@
 	7850 5300 7850 5400
 $Comp
-L GND #PWR035
+L GND #PWR029
 U 1 1 537E6A4E
 P 7850 5400
-F 0 "#PWR035" H 7850 5400 30  0001 C CNN
+F 0 "#PWR029" H 7850 5400 30  0001 C CNN
 F 1 "GND" H 7850 5330 30  0001 C CNN
 F 2 "~" H 7850 5400 60  0000 C CNN
@@
 	7850 6100 7850 6200
 $Comp
-L GND #PWR036
+L GND #PWR030
 U 1 1 537E6A65
 P 7850 6200
-F 0 "#PWR036" H 7850 6200 30  0001 C CNN
+F 0 "#PWR030" H 7850 6200 30  0001 C CNN
 F 1 "GND" H 7850 6130 30  0001 C CNN
 F 2 "~" H 7850 6200 60  0000 C CNN
@@
 	9500 5350 9500 5450
 $Comp
-L GND #PWR037
+L GND #PWR031
 U 1 1 537E6A80
 P 9500 5450
-F 0 "#PWR037" H 9500 5450 30  0001 C CNN
+F 0 "#PWR031" H 9500 5450 30  0001 C CNN
 F 1 "GND" H 9500 5380 30  0001 C CNN
 F 2 "~" H 9500 5450 60  0000 C CNN
@@
 	9500 6150 9500 6250
 $Comp
-L GND #PWR038
+L GND #PWR032
 U 1 1 537E6A97
 P 9500 6250
-F 0 "#PWR038" H 9500 6250 30  0001 C CNN
+F 0 "#PWR032" H 9500 6250 30  0001 C CNN
 F 1 "GND" H 9500 6180 30  0001 C CNN
 F 2 "~" H 9500 6250 60  0000 C CNN
@@
 	6400 1800 5850 1800
 $Comp
-L GND #PWR039
+L GND #PWR033
 U 1 1 537E6E27
 P 6650 1500
-F 0 "#PWR039" H 6650 1500 30  0001 C CNN
+F 0 "#PWR033" H 6650 1500 30  0001 C CNN
 F 1 "GND" H 6650 1430 30  0001 C CNN
 F 2 "~" H 6650 1500 60  0000 C CNN
@@
 	4750 1000 4750 1500
 $Comp
-L GND #PWR040
+L GND #PWR034
 U 1 1 537E72EF
 P 4650 1700
-F 0 "#PWR040" H 4650 1700 30  0001 C CNN
+F 0 "#PWR034" H 4650 1700 30  0001 C CNN
 F 1 "GND" H 4650 1630 30  0001 C CNN
 F 2 "~" H 4650 1700 60  0000 C CNN
@@
 Connection ~ 7800 1450
 $Comp
-L GND #PWR041
+L GND #PWR035
 U 1 1 538D7812
 P 7800 2150
-F 0 "#PWR041" H 7800 2150 30  0001 C CNN
+F 0 "#PWR035" H 7800 2150 30  0001 C CNN
 F 1 "GND" H 7800 2080 30  0001 C CNN
 F 2 "~" H 7800 2150 60  0000 C CNN
@@
 $EndComp
 $Comp
-L GND #PWR042
+L GND #PWR036
 U 1 1 538D791A
 P 9500 2250
-F 0 "#PWR042" H 9500 2250 30  0001 C CNN
+F 0 "#PWR036" H 9500 2250 30  0001 C CNN
 F 1 "GND" H 9500 2180 30  0001 C CNN
 F 2 "~" H 9500 2250 60  0000 C CNN
@@
 $EndComp
 $Comp
-L GND #PWR043
+L GND #PWR037
 U 1 1 53924614
 P 8150 4000
-F 0 "#PWR043" H 8150 4000 30  0001 C CNN
+F 0 "#PWR037" H 8150 4000 30  0001 C CNN
 F 1 "GND" H 8150 3930 30  0001 C CNN
 F 2 "~" H 8150 4000 60  0000 C CNN
@@
 	8150 4000 8150 3950
 $Comp
-L GND #PWR044
+L GND #PWR038
 U 1 1 5392461B
 P 9450 4000
-F 0 "#PWR044" H 9450 4000 30  0001 C CNN
+F 0 "#PWR038" H 9450 4000 30  0001 C CNN
 F 1 "GND" H 9450 3930 30  0001 C CNN
 F 2 "~" H 9450 4000 60  0000 C CNN
@@
 $EndComp
 $Comp
-L GND #PWR045
+L GND #PWR039
 U 1 1 539A1B02
 P 3200 5250
-F 0 "#PWR045" H 3200 5250 30  0001 C CNN
+F 0 "#PWR039" H 3200 5250 30  0001 C CNN
 F 1 "GND" H 3200 5180 30  0001 C CNN
 F 2 "~" H 3200 5250 60  0000 C CNN
@@
 Y
 $Comp
-L GND #PWR046
+L GND #PWR040
 U 1 1 539A1B17
 P 2000 5250
-F 0 "#PWR046" H 2000 5250 30  0001 C CNN
+F 0 "#PWR040" H 2000 5250 30  0001 C CNN
 F 1 "GND" H 2000 5180 30  0001 C CNN
 F 2 "~" H 2000 5250 60  0000 C CNN
@@
 $EndComp
 $Comp
-L GND #PWR047
+L GND #PWR041
 U 1 1 539A1B1D
 P 3000 5250
-F 0 "#PWR047" H 3000 5250 30  0001 C CNN
+F 0 "#PWR041" H 3000 5250 30  0001 C CNN
 F 1 "GND" H 3000 5180 30  0001 C CNN
 F 2 "~" H 3000 5250 60  0000 C CNN
@@
 Wire Wire Line
 	5100 6950 5100 7400
-$Comp
-L GND #PWR048
-U 1 1 539C8F1D
-P 5100 7400
-F 0 "#PWR048" H 5100 7400 30  0001 C CNN
-F 1 "GND" H 5100 7330 30  0001 C CNN
-F 2 "~" H 5100 7400 60  0000 C CNN
-F 3 "~" H 5100 7400 60  0000 C CNN
-	1    5100 7400
-	1    0    0    -1
-$EndComp
 Wire Wire Line
 	3100 6700 3000 6700
@@
 	7750 3350 7750 3400
 $Comp
-L GND #PWR049
+L GND #PWR042
 U 1 1 539D1ECC
 P 7750 3400
-F 0 "#PWR049" H 7750 3400 30  0001 C CNN
+F 0 "#PWR042" H 7750 3400 30  0001 C CNN
 F 1 "GND" H 7750 3330 30  0001 C CNN
 F 2 "~" H 7750 3400 60  0000 C CNN
@@
 $EndComp
 $Comp
-L GND #PWR050
+L GND #PWR043
 U 1 1 53A8A584
 P 3200 2900
-F 0 "#PWR050" H 3200 2900 30  0001 C CNN
+F 0 "#PWR043" H 3200 2900 30  0001 C CNN
 F 1 "GND" H 3200 2830 30  0001 C CNN
 F 2 "~" H 3200 2900 60  0000 C CNN
@@
 Z
 $Comp
-L GND #PWR051
+L GND #PWR044
 U 1 1 53A8A599
 P 2000 2900
-F 0 "#PWR051" H 2000 2900 30  0001 C CNN
+F 0 "#PWR044" H 2000 2900 30  0001 C CNN
 F 1 "GND" H 2000 2830 30  0001 C CNN
 F 2 "~" H 2000 2900 60  0000 C CNN
@@
 $EndComp
 $Comp
-L GND #PWR052
+L GND #PWR045
 U 1 1 53A8A59F
 P 3000 2900
-F 0 "#PWR052" H 3000 2900 30  0001 C CNN
+F 0 "#PWR045" H 3000 2900 30  0001 C CNN
 F 1 "GND" H 3000 2830 30  0001 C CNN
 F 2 "~" H 3000 2900 60  0000 C CNN
@@
 	1    0    0    -1
 $EndComp
+Wire Wire Line
+	4500 7400 5200 7400
+Connection ~ 5100 7400
+Text GLabel 5200 7400 2    60   UnSpc ~ 0
+AGND
 $EndSCHEMATC

Commit message: Pin swap. Route.
Connections:
- net D2: now also C18.1, R27.1; no longer C15.1, R24.1
- net D3: now also C15.1, R24.1; no longer C18.1, R27.1
- net D25 renamed D15
Changed lines of the file:
@@
 Text Label 8550 5700 2    60   ~ 0
 Ymax
-Text GLabel 7750 4900 0    50   Input ~ 0
+Text GLabel 9400 5750 0    50   Input ~ 0
 D2
 Text GLabel 7750 5700 0    50   Input ~ 0
-D25
+D15
 $Comp
 L R R24
@@
 Text GLabel 9400 4950 0    50   Input ~ 0
 D14
-Text GLabel 9400 5750 0    50   Input ~ 0
+Text GLabel 7750 4900 0    50   Input ~ 0
 D3
 $Comp
